File: PMOD-100BASET1.kicad_sch (KiCad schematic)
At the start: 115 parts, among them J1 Conn_01x02, J2 RB1-125B8G1A, J3 2304372-1, J4 Conn_01x02, J5 Tag Connect SWD, P1 USB_C_Plug_USB2.0, Q1 AO3401A, Q2 AO3400A, Q3 AO3401A, Q4 AO3400A, SW1 Reset, SW2 Boot, U1 AP1117-33, U2 STM32F072CBTx, U3 24LC16, U4 DP83TC813RRHFRQ1, U5 LAN8720A, Y1 25MHz

Commit message: [doc] added readme; updated files to Kicad V8
Parts:
- removed C1, C10, C17, C2, C22, C28: 4.7u, Capacitor_SMD:C_0603_1608Metric, symbol Device:C
- removed C12, C14, C23, C24, C27, C29, C3, C30, C31, C32, C6: 100n, Capacitor_SMD:C_0603_1608Metric, symbol Device:C
- removed C15, C4, C5: 10p, Capacitor_SMD:C_0603_1608Metric, symbol Device:C
- removed C19: 470p, Capacitor_SMD:C_0603_1608Metric, symbol Device:C
- removed C21: 20p, Capacitor_SMD:C_0603_1608Metric, symbol Device:C
- removed D1: 1N5819, Diode_SMD:D_SOD-323, symbol Diode:1N5819
- removed FB2: 100@100M, Resistor_SMD:R_0805_2012Metric, symbol Device:FerriteBead_Small
- removed H1: MountingHole, MountingHole:MountingHole_2.5mm, symbol Mechanical:MountingHole
- removed J2: RB1-125B8G1A, Connector_RJ:RJ45_UDE_RB1-125B8G1A, symbol Connector:RB1-125B8G1A
- removed J4: Conn_01x02, Connector_JST:JST_XH_B2B-XH-A_1x02_P2.50mm_Vertical, symbol Connector_Generic:Conn_01x02
- removed J5: Tag Connect SWD, Connector:Tag-Connect_TC2030-IDC-FP_2x03_P1.27mm_Vertical, symbol Connector_Generic:Conn_02x03_Odd_Even
- removed LD1: YELLOW, LED_SMD:LED_0603_1608Metric, symbol Device:LED
- removed LD2: RED, LED_SMD:LED_0603_1608Metric, symbol Device:LED
- removed P1: USB_C_Plug_USB2.0, Connector_USB:USB_C_Receptacle_GCT_USB4085, symbol Connector:USB_C_Plug_USB2.0
- removed PMOD2: PMOD-Device-x2-Type-1A-GPIO, pmod-conn_6x2:pmod_pin_array_6x2, symbol pmod:PMOD-Device-x2-Type-1A-GPIO
- removed Q1, Q3: AO3401A, Package_TO_SOT_SMD:SOT-23, symbol Device:Q_PMOS_GSD
- removed Q2, Q4: AO3400A, Package_TO_SOT_SMD:SOT-23, symbol Transistor_FET:AO3400A
- removed R10, R11, R18, R19, R22, R38, R45, R47, R8, R9: 1k, Resistor_SMD:R_0603_1608Metric, symbol Device:R
- removed R17, R24, R25, R26, R27, R34: 10, Resistor_SMD:R_0603_1608Metric, symbol Device:R
- removed R20, R21, R23, R43, R5, R6: 2.4k, Resistor_SMD:R_0603_1608Metric, symbol Device:R
- removed R29: 0, Resistor_SMD:R_0603_1608Metric, symbol Device:R
- removed R31, R32, R33, R36: 49.9, Resistor_SMD:R_0603_1608Metric, symbol Device:R
- removed R37: 12k, Resistor_SMD:R_0603_1608Metric, symbol Device:R
- removed R7: 5.1k, Resistor_SMD:R_0603_1608Metric, symbol Device:R
- removed SW1: Reset, Button_Switch_SMD:SW_Push_1P1T_NO_6x6mm_H9.5mm, symbol Switch:SW_Push
- removed SW2: Boot, Button_Switch_SMD:SW_Push_1P1T_NO_6x6mm_H9.5mm, symbol Switch:SW_Push
- removed U1: AP1117-33, Package_TO_SOT_SMD:SOT-223-3_TabPin2, symbol Regulator_Linear:AP1117-33
- removed U2: STM32F072CBTx, Package_QFP:LQFP-48_7x7mm_P0.5mm, symbol MCU_ST_STM32F0:STM32F072CBTx
- removed U3: 24LC16, Package_SO:SOIC-8_3.9x4.9mm_P1.27mm, symbol Memory_EEPROM:24LC16
- removed U5: LAN8720A, Package_DFN_QFN:QFN-24-1EP_4x4mm_P0.5mm_EP2.6x2.6mm, symbol Interface_Ethernet:LAN8720A
- removed Y1: 25MHz, Crystal:Crystal_SMD_3225-4Pin_3.2x2.5mm, symbol Device:Crystal_GND24
- added J8, J9: Conn_01x03, Connector_PinHeader_2.54mm:PinHeader_1x04_P2.54mm_Vertical, symbol Connector_Generic:Conn_01x04
- added JP1, JP2: SolderJumper_3_Open, Jumper:SolderJumper-3_P1.3mm_Open_RoundedPad1.0x1.5mm, symbol Jumper:SolderJumper_3_Open
- J1, J3, R40: now not fitted
- LD3: value BLUE -> WHITE; LCSC C72041 -> C2290
- R1: value 2.4k -> 4.7k; LCSC C22940 -> C23162
- R2, R4: value 2.4k -> 9.1k; LCSC C22940 -> C23260
- R3: value 10 -> 4.7k; LCSC C22859 -> C23162
Connections:
- net U1_TX is gone; now on net RXER: R3.1
- net VDD_T1 is gone; now on net +3V3: C18.2, C7.2, C8.2, FB1.1, R30.1, R39.1
- net +3V3: now also J8.1 (Pin_1), J9.1 (Pin_1); no longer R1.2, R2.2, R4.2
- net GND: now also C33.2, C34.2, L4.1, L5.1, J8.2 (Pin_2), J9.4 (Pin_4)
- net MDC_T1: now also J9.3 (Pin_3)
- net MDIO_T1: now also J9.2 (Pin_2)
- net RST_T1: now also PMOD1.10 (IOB3)
- net RX_D3: no longer R35.2
- net RX_DV: now also R1.1
- net VDDIO: now also R2.2, R4.2, JP1.1 (A), JP2.1 (A)
- net at U4.13 (XI): now also R35.1
- net RXER: now reaches U4.21 (RXER)
- net V_P: now reaches C33.1, C34.1, L2.1, L3.1
- net V_P: now also J8.3 (Pin_3), J8.4 (Pin_4)
- net REFCLK_PMOD renamed REFCLK
- net REFCLK: now also R35.2; no longer R35.1
- net SCL: no longer names the net of R4.1
- net SCL: now also JP2.3 (B)
- net SDA: no longer names the net of R2.1
- net SDA: now also JP1.3 (B)
- removed net TRX_STM: PMOD1.10 (IOB3), R1.1, R3.2
- new net: JP1.2 (C), R1.2
- new net: JP2.2 (C), R3.2
- no-connect marks 13 -> 5
Other:
- note added: "MAC[0]=0"
- note removed: "100BASE-T PHY"
- note removed: "100BASE-T Supply"
- note removed: "3V3 Supply"
- note removed: "Configuration MCU"
- note removed: "I2C2"
- note removed: "I2C: 0b1010000"
- note removed: "MAC[0]=1"
- note removed: "Mechanical"
- note removed: "PHYADD=1"
- note removed: "SLAVE MODE"
- note removed: "U1_RX"
- note removed: "int. PD: REG ON int. PU: REFCLK IN"
- moved on the sheet: C11, C13, C16, C18, C20, C33, C34, C7, C8, C9, FB1, L2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
